File: Hardware/Neko_Wireless_Transmission.kicad_pcb (KiCad board)
At the start: 2 copper layers, 25 x 25 mm, 48 parts, among them IC1 W25Q32JVSSIQ, IC2 ESP32-D0WD, IC3 IPS6404L-SQ-SPN, J1 OV2640, Q1 AO3401A, U1 XC6206P282MR, U2 XC6206P122MR, Y1 YSX321SL_40Mhz

Commit message: Finished PCB Layout
Routing:
- net /CSI_MCLK: track 16.4 -> 17.7 mm
- net /CSI_HSYNC: track 16.4 -> 17.1 mm
- net /SDIO_CMD: track 16.5 -> 17.0 mm
- net +3.3V: track 63.2 -> 63.7 mm

Commit message: Update PCB V3.2
Parts:
- added ?: , SamacSys_Parts:nya_mini, F.Cu at (47.3, 71.1)
Routing:
- net GND: vias 146 -> 124
